File: PCB/HoneyBee/newschematic.kicad_sch (KiCad schematic)
At the start: 42 parts, among them J1 S2B-PH-K-SLFSN, J2 10104110-0001LF, M1 Motor_DC, M2 Motor_DC, M3 Motor_DC, M4 Motor_DC, M5 Motor_DC, M6 Motor_DC, Q1 IRLML2502TRPbF, Q2 IRLML2502TRPbF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

Commit message: Updated BOM, Changed Components
Added "Price" and "DigiKey" to BOM
Changed out of stock components and non-Cut Reel components.
Parts:
- removed C11: 10 uF, Capacitor_SMD:C_0603_1608Metric_Pad1.08x0.95mm_HandSolder, symbol Device:C
- removed U2: LM2940HS-3.3, Package_TO_SOT_SMD:SOT-223-3_TabPin2, symbol Regulator_Linear:AZ1117-3.3
- added R10: 52.3K, Resistor_SMD:R_0603_1608Metric_Pad0.98x0.95mm_HandSolder, symbol Device:R
- added R9: 30.1K, Resistor_SMD:R_0603_1608Metric_Pad0.98x0.95mm_HandSolder, symbol Device:R
- added U2: TPS73733DCQR, Package_TO_SOT_SMD:SOT-23-5, symbol Regulator_Linear:TPS73018DBV
- C1, C10, C13, C14, C17, C18, C4, C5, C9: DigiKey (none) -> https://www.digikey.com/en/products/detail/kemet/C0603C104K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; Unit Price (none) -> 0.08
- C12: DigiKey (none) -> https://www.digikey.com/en/products/detail/murata-electroni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; Unit Price (none) -> 0.13
- C2, C3, C8: DigiKey (none) -> https://www.digikey.com/en/products/detail/kemet/C0603C105K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; Unit Price (none) -> 0.08
- C6: DigiKey (none) -> https://www.digikey.com/en/products/detail/kemet/C0603C106M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; Unit Price (none) -> 0.28
- C7: footprint Capacitor_SMD:C_0603_1608Metric_Pad1.08x0.95mm_HandSolder -> Capacitor_SMD:C_0805_2012Metric_Pad1.18x1.45mm_HandSolder; DigiKey (none) -> https://www.digikey.com/en/products/detail/murata-electroni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; Unit Price (none) -> 0.53
- CR1, CR2, CR3: value PMEG2010AEB -> SS24FL; footprint Diode_SMD:D_SOD-523 -> Diode_SMD:D_SOD-123F; DigiKey (none) -> https://www.digikey.com/en/products/detail/onsemi/SS24FL/53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; Unit Price (none) -> 0.27
- J1: DigiKey (none) -> https://www.digikey.com/en/products/detail/jst-sales-americ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; Unit Price (none) -> 0.11
- J2: DigiKey (none) -> https://www.digikey.com/en/products/detail/amphenol-cs-fci/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; Unit Price (none) -> 0.81
- M1, M2: Unit Price (none) -> 6.88
- M3, M4, M5, M6: Unit Price (none) -> 6
- Q1, Q2: Unit Price (none) -> 0.14
- R1, R2, R3, R4, R5, R6, R7, R8: DigiKey (none) -> https://www.digikey.com/en/products/detail/yageo/RC0603FR-0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; Unit Price (none) -> 0.10
- U1: DigiKey (none) -> https://www.digikey.com/en/products/detail/microchip-techno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; Unit Price (none) -> 4.25
- U3: DigiKey (none) -> https://www.digikey.com/en/products/detail/omron-electronic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; Unit Price (none) -> 0.90
- U6: DigiKey (none) -> https://www.digikey.com/en/products/detail/bosch-sensortec/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; Unit Price (none) -> 3.27
- U8: DigiKey (none) -> https://www.digikey.com/en/products/detail/toshiba-semicond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; Unit Price (none) -> 1.82
Connections:
- net +3.3V: now also R10.1, U2.5 (OUT)
- net GND: now also R9.2, U2.2 (GND)
- net at C1.2, C18.1, C5.2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: now also U2.1 (IN), U2.3 (EN)
- new net: R10.2, R9.1, U2.4 (NR)
Other:
- moved on the sheet: C12

Commit message: Small Tweaks
Parts:
- U2: footprint Package_TO_SOT_SMD:SOT-23-5 -> Package_TO_SOT_SMD:SOT-223-6_TabPin3
Changed lines of the file:
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@@
 			)
 		)
-		(property "Footprint" "Package_TO_SOT_SMD:SOT-23-5"
+		(property "Footprint" "Package_TO_SOT_SMD:SOT-223-6_TabPin3"
 			(at 115.57 43.815 0)
 			(effects
