File: PCB/HoneyBee/newschematic.kicad_pcb (KiCad board)
At the start: 4 copper layers, 50 x 50 mm, 46 parts, among them J1 S2B-PH-K-SLFSN, J2 10104110-0001LF, J3 01x05_MountingPin, M1 Motor_DC, M2 Motor_DC, M3 Motor_DC, M4 Motor_DC, M5 Motor_DC, M6 Motor_DC, Q1 IRLML2502TRPbF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

Commit message: Removed regulator resistors, Added capacitor
Parts:
- removed R10: 52.3K, Resistor_SMD:R_0603_1608Metric_Pad0.98x0.95mm_HandSolder
- removed R9: 30.1K, Resistor_SMD:R_0603_1608Metric_Pad0.98x0.95mm_HandSolder
- added C1: 0.1 uF, Capacitor_SMD:C_0603_1608Metric_Pad1.08x0.95mm_HandSolder, B.Cu at (87.8, 67.1)
- turned CR1 to 0 degrees
- turned CR3 to 0 degrees
Connections:
- CR1 pad 1: Net-(M1--) -> +BATT
- CR1 pad 2: +BATT -> Net-(M1--)
- CR3 pad 1: Net-(M2--) -> +BATT
- CR3 pad 2: +BATT -> Net-(M2--)
- U2 pad 4: Net-(U2-NR) -> GND
Routing:
- net Net-(U2-NR): track 5.78 -> 0.00 mm
- net GND: track 55.4 -> 60.6 mm
- net +3.3V: track 28.0 -> 26.6 mm, vias 23 -> 22
